File: PCBs/LASK4/LASK4/LASK4.kicad_sch (KiCad schematic)
At the start: 16 parts

Commit message: LASK4 Update
Updated LASK4 PCB and pertaining documents.
Parts:
- added H5, H6, H7: MountingHole_Pad, MountingHole:MountingHole_2.2mm_M2_DIN965_Pad, symbol Mechanical:MountingHole_Pad
- gave numbers to parts that had none: 12
- renumbered Down to Down1, Select to Select1, Start to Start1, Up to Up1
Connections:
- net GND: now also H5.1, H6.1, H7.1

Commit message: LASK4V2
Parts:
- added Switch1: SW_SPDT, Connector_PinHeader_2.54mm:PinHeader_1x03_P2.54mm_Vertical, symbol Switch:SW_SPDT
Connections:
- net +5V: now also Switch1.2 (B); no longer U5.1 (VIN), U5.6 (OUT-5V)
- new net BatterPowered: Switch1.1 (A), U5.6 (OUT-5V)
- new net ChargingMode: Switch1.3 (C), U5.1 (VIN)
Changed lines of the file:
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@@
   (junction (at 156.21 78.74) (diameter 0) (color 0 0 0 0)
   )
-  (junction (at 139.7 101.6) (diameter 0) (color 0 0 0 0)
-  )
   (junction (at 248.92 97.79) (diameter 0) (color 0 0 0 0)
   )
@@
   (junction (at 105.41 78.74) (diameter 0) (color 0 0 0 0)
   )
-  (junction (at 142.24 109.22) (diameter 0) (color 0 0 0 0)
-  )
   (junction (at 138.43 78.74) (diameter 0) (color 0 0 0 0)
   )
@@
     (stroke (width 0) (type default) (color 0 0 0 0))
   )
-  (wire (pts (xy 139.7 101.6) (xy 146.05 101.6))
-    (stroke (width 0) (type default) (color 0 0 0 0))
-  )
   (wire (pts (xy 250.19 77.47) (xy 245.11 77.47))
     (stroke (width 0) (type default) (color 0 0 0 0))
@@
     (stroke (width 0) (type default) (color 0 0 0 0))
   )
-  (wire (pts (xy 138.43 111.76) (xy 146.05 111.76))
+  (wire (pts (xy 138.43 111.76) (xy 153.67 111.76))
     (stroke (width 0) (type default) (color 0 0 0 0))
   )
@@
     (stroke (width 0) (type default) (color 0 0 0 0))
   )
+  (wire (pts (xy 146.05 93.98) (xy 151.13 93.98))
+    (stroke (width 0) (type default) (color 0 0 0 0))
+  )
   (wire (pts (xy 73.66 53.34) (xy 107.95 53.34))
     (stroke (width 0) (type default) (color 0 0 0 0))
@@
     (stroke (width 0) (type default) (color 0 0 0 0))
   )
-  (wire (pts (xy 138.43 109.22) (xy 142.24 109.22))
+  (wire (pts (xy 138.43 109.22) (xy 146.05 109.22))
     (stroke (width 0) (type default) (color 0 0 0 0))
   )
@@
     (stroke (width 0) (type default) (color 0 0 0 0))
   )
-  (wire (pts (xy 138.43 114.3) (xy 139.7 114.3))
+  (wire (pts (xy 138.43 114.3) (xy 138.43 119.38))
     (stroke (width 0) (type default) (color 0 0 0 0))
   )
@@
     (stroke (width 0) (type default) (color 0 0 0 0))
   )
+  (wire (pts (xy 146.05 101.6) (xy 138.43 101.6))
+    (stroke (width 0) (type default) (color 0 0 0 0))
+  )
   (wire (pts (xy 245.11 100.33) (xy 259.08 100.33))
     (stroke (width 0) (type default) (color 0 0 0 0))
   )
-  (wire (pts (xy 142.24 109.22) (xy 146.05 109.22))
-    (stroke (width 0) (type default) (color 0 0 0 0))
-  )
   (wire (pts (xy 208.28 80.01) (xy 217.17 80.01))
     (stroke (width 0) (type default) (color 0 0 0 0))
@@
     (stroke (width 0) (type default) (color 0 0 0 0))
   )
-  (wire (pts (xy 142.24 104.14) (xy 142.24 109.22))
-    (stroke (width 0) (type default) (color 0 0 0 0))
-  )
   (wire (pts (xy 138.43 78.74) (xy 156.21 78.74))
     (stroke (width 0) (type default) (color 0 0 0 0))
@@
     (stroke (width 0) (type default) (color 0 0 0 0))
   )
-  (wire (pts (xy 139.7 114.3) (xy 139.7 101.6))
-    (stroke (width 0) (type default) (color 0 0 0 0))
-  )
   (wire (pts (xy 208.28 82.55) (xy 217.17 82.55))
     (stroke (width 0) (type default) (color 0 0 0 0))
@@
     (stroke (width 0) (type default) (color 0 0 0 0))
   )
-  (wire (pts (xy 138.43 104.14) (xy 142.24 104.14))
+  (wire (pts (xy 138.43 104.14) (xy 146.05 104.14))
     (stroke (width 0) (type default) (color 0 0 0 0))
   )
@@
     (stroke (width 0) (type default) (color 0 0 0 0))
   )
-  (wire (pts (xy 138.43 101.6) (xy 139.7 101.6))
-    (stroke (width 0) (type default) (color 0 0 0 0))
-  )
   (wire (pts (xy 172.72 78.74) (xy 172.72 80.01))
     (stroke (width 0) (type default) (color 0 0 0 0))
@@
     (effects (font (size 1.27 1.27)) (justify left bottom))
   )
+  (label "ChargingMode" (at 161.29 96.52 0)
+    (effects (font (size 1.27 1.27)) (justify left bottom))
+  )
   (label "SDA34" (at 176.53 106.68 0)
     (effects (font (size 1.27 1.27)) (justify left bottom))
@@
     (effects (font (size 1.27 1.27)) (justify left bottom))
   )
+  (label "BatGND" (at 146.05 104.14 0)
+    (effects (font (size 1.27 1.27)) (justify left bottom))
+  )
+  (label "BatterPowered" (at 146.05 101.6 0)
+    (effects (font (size 1.27 1.27)) (justify left bottom))
+  )
   (label "Down" (at 119.38 135.89 0)
     (effects (font (size 1.27 1.27)) (justify left bottom))
   )
+  (label "ChargingMode" (at 138.43 119.38 0)
+    (effects (font (size 1.27 1.27)) (justify left bottom))
+  )
   (label "Select" (at 138.43 135.89 0)
     (effects (font (size 1.27 1.27)) (justify left bottom))
@@
   )
   (label "Select" (at 208.28 82.55 0)
+    (effects (font (size 1.27 1.27)) (justify left bottom))
+  )
+  (label "BatterPowered" (at 161.29 91.44 0)
     (effects (font (size 1.27 1.27)) (justify left bottom))
   )
@@
     (pin "3")
   )
-  (symbol (lib_id "power:+5V") (at 146.05 101.6 0) (unit 1)
-    (in_bom yes) (on_board yes) (fields_autoplaced)
-    (property "Reference" "#PWR0103" (id 0) (at 146.05 105.41 0)
-      (effects (font (size 1.27 1.27)) hide)
-    )
-    (property "Value" "+5V" (id 1) (at 146.05 96.52 0))
-    (property "Footprint" "" (id 2) (at 146.05 101.6 0)
-      (effects (font (size 1.27 1.27)) hide)
-    )
-    (property "Datasheet" "" (id 3) (at 146.05 101.6 0)
+  (symbol (lib_id "power:+5V") (at 146.05 93.98 0) (unit 1)
+    (in_bom yes) (on_board yes)
+    (property "Reference" "#PWR0103" (id 0) (at 146.05 97.79 0)
+      (effects (font (size 1.27 1.27)) hide)
+    )
+    (property "Value" "+5V" (id 1) (at 146.05 87.63 0))
+    (property "Footprint" "" (id 2) (at 146.05 93.98 0)
+      (effects (font (size 1.27 1.27)) hide)
+    )
+    (property "Datasheet" "" (id 3) (at 146.05 93.98 0)
       (effects (font (size 1.27 1.27)) hide)
     )
@@
     (pin "3")
   )
+  (symbol (lib_id "Switch:SW_SPDT") (at 156.21 93.98 0) (unit 1)
+    (in_bom yes) (on_board yes) (fields_autoplaced)
+    (property "Reference" "Switch1" (id 0) (at 156.21 86.36 0))
+    (property "Value" "SW_SPDT" (id 1) (at 156.21 88.9 0))
+    (property "Footprint" "Connector_PinHeader_2.54mm:PinHeader_1x03_P2.54mm_Vertical" (id 2) (at 156.21 93.98 0)
+      (effects (font (size 1.27 1.27)) hide)
+    )
+    (property "Datasheet" "~" (id 3) (at 156.21 93.98 0)
+      (effects (font (size 1.27 1.27)) hide)
+    )
+    (pin "1")
+    (pin "2")
+    (pin "3")
+  )
   (symbol (lib_id "OpenMuscleLibrary:Hall-49E") (at 139.7 45.72 0) (unit 1)
     (in_bom yes) (on_board yes)
@@
     (pin "1")
   )
-  (symbol (lib_id "power:GND") (at 146.05 111.76 0) (unit 1)
-    (in_bom yes) (on_board yes) (fields_autoplaced)
-    (property "Reference" "#PWR0104" (id 0) (at 146.05 118.11 0)
-      (effects (font (size 1.27 1.27)) hide)
-    )
-    (property "Value" "GND" (id 1) (at 146.05 116.84 0))
-    (property "Footprint" "" (id 2) (at 146.05 111.76 0)
-      (effects (font (size 1.27 1.27)) hide)
-    )
-    (property "Datasheet" "" (id 3) (at 146.05 111.76 0)
+  (symbol (lib_id "power:GND") (at 153.67 111.76 0) (unit 1)
+    (in_bom yes) (on_board yes) (fields_autoplaced)
+    (property "Reference" "#PWR0104" (id 0) (at 153.67 118.11 0)
+      (effects (font (size 1.27 1.27)) hide)
+    )
+    (property "Value" "GND" (id 1) (at 153.67 116.84 0))
+    (property "Footprint" "" (id 2) (at 153.67 111.76 0)
+      (effects (font (size 1.27 1.27)) hide)
+    )
+    (property "Datasheet" "" (id 3) (at 153.67 111.76 0)
       (effects (font (size 1.27 1.27)) hide)
     )
@@
       (reference "Start1") (unit 1) (value "SW_Push") (footprint "Button_Switch_THT:SW_PUSH_6mm")
     )
+    (path "/d70251a2-958d-427d-bf99-1b80f1a78708"
+      (reference "Switch1") (unit 1) (value "SW_SPDT") (footprint "Connector_PinHeader_2.54mm:PinHeader_1x03_P2.54mm_Vertical")
+    )
     (path "/36d8f133-3da2-4a49-9e47-97e46dfb5ab4"
